Commit message: Created arm mass sims base hw xacro and Unit D no arms xacro

File: model/robots/common/xacro/arm/arm.xacro (robot description, xacro)
@@ -152,4 +152,19 @@
     </xacro:revolute_joint_ex>
   </xacro:macro>
+    <xacro:macro name="make_lower_arm_mass_sim" params="prefix reflect lower_arm_root_link">
+    <xacro:standard_link name="${ForearmLinkName}"
+                    mass="${ForearmYawLinkMass}"
+                    origin_xyz="${ForearmYawLinkComPosition}"
+                    ixx="${ForearmYawLinkInertia_IXX}" ixy="${ForearmYawLinkInertia_IXY}" ixz="${ForearmYawLinkInertia_IXZ}"
+                    iyy="${ForearmYawLinkInertia_IYY}" iyz="${ForearmYawLinkInertia_IYZ}" izz="${ForearmYawLinkInertia_IZZ}"
+                    origin_rpy="0 0 0"
+                    visual_mesh="${mesh_root}/arms/${prefix}_elbow_mass_sim.dae"
+                    collision_mesh="${mesh_root}/arms/${prefix}_elbow_mass_sim.dae" />
+    <xacro:fixed_joint jointName="${ForearmYawJointName}"
+                          parent="${lower_arm_root_link}" child="${ForearmLinkName}"
+                          origin_xyz="${ForearmYawFrameOrigin_X} ${ForearmYawFrameOrigin_Y} ${ForearmYawFrameOrigin_Z}"
+                          origin_rpy="${ForearmYawFrameOrientation_Roll} ${ForearmYawFrameOrientation_Pitch} ${ForearmYawFrameOrientation_Yaw}">
+    </xacro:fixed_joint>
+  </xacro:macro>
   <xacro:macro name="make_arm" params="prefix reflect arm_root_link">
     <xacro:make_upper_arm prefix="${prefix}" reflect="${reflect}" upper_arm_root_link="${arm_root_link}" />
@@ -158,4 +173,8 @@
   <xacro:macro name="make_arm_no_hands" params="prefix reflect arm_root_link">
     <xacro:make_upper_arm prefix="${prefix}" reflect="${reflect}" upper_arm_root_link="${arm_root_link}" />
+  </xacro:macro>
+  <xacro:macro name="make_arm_mass_sims" params="prefix reflect arm_root_link">
+    <xacro:make_upper_arm prefix="${prefix}" reflect="${reflect}" upper_arm_root_link="${arm_root_link}" />
+    <xacro:make_lower_arm_mass_sim prefix="${prefix}" reflect="${reflect}" lower_arm_root_link="${ElbowPitchLinkName}" />
   </xacro:macro>
   <xacro:macro name="arm_transmissions_hw" params="prefix reflect">

Commit message: Created simulation version of arm mass sims Valkyrie

File: model/robots/common/xacro/arm/arm.xacro (robot description, xacro)
@@ -154,8 +154,8 @@
     <xacro:macro name="make_lower_arm_mass_sim" params="prefix reflect lower_arm_root_link">
     <xacro:standard_link name="${ForearmLinkName}"
-                    mass="${ForearmYawLinkMass}"
-                    origin_xyz="${ForearmYawLinkComPosition}"
-                    ixx="${ForearmYawLinkInertia_IXX}" ixy="${ForearmYawLinkInertia_IXY}" ixz="${ForearmYawLinkInertia_IXZ}"
-                    iyy="${ForearmYawLinkInertia_IYY}" iyz="${ForearmYawLinkInertia_IYZ}" izz="${ForearmYawLinkInertia_IZZ}"
+                    mass="${ForearmMassSimLinkMass}"
+                    origin_xyz="${ForearmMassSimComPosition}"
+                    ixx="${ForearmMassSimInertia_IXX}" ixy="${ForearmMassSimInertia_IXY}" ixz="${ForearmMassSimInertia_IXZ}"
+                    iyy="${ForearmMassSimInertia_IYY}" iyz="${ForearmMassSimInertia_IYZ}" izz="${ForearmMassSimInertia_IZZ}"
                     origin_rpy="0 0 0"
                     visual_mesh="${mesh_root}/arms/${prefix}_elbow_mass_sim.dae"
@@ -163,6 +163,6 @@
     <xacro:fixed_joint jointName="${ForearmYawJointName}"
                           parent="${lower_arm_root_link}" child="${ForearmLinkName}"
-                          origin_xyz="${ForearmYawFrameOrigin_X} ${ForearmYawFrameOrigin_Y} ${ForearmYawFrameOrigin_Z}"
-                          origin_rpy="${ForearmYawFrameOrientation_Roll} ${ForearmYawFrameOrientation_Pitch} ${ForearmYawFrameOrientation_Yaw}">
+                          origin_xyz="${ForearmMassSimFrameOrigin_X} ${ForearmMassSimFrameOrigin_Y} ${ForearmMassSimFrameOrigin_Z}"
+                          origin_rpy="${ForearmMassSimFrameOrientation_Roll} ${ForearmMassSimFrameOrientation_Pitch} ${ForearmMassSimFrameOrientation_Yaw}">
     </xacro:fixed_joint>
   </xacro:macro>

File: model/robots/common/xacro/arm/frame_parameters.xacro (robot description, xacro)
@@ -31,4 +31,10 @@
   <xacro:property name="ForearmYawFrameOrientation_Pitch" value="0.0"/>
   <xacro:property name="ForearmYawFrameOrientation_Yaw" value="0.0"/>
+  <xacro:property name="ForearmMassSimFrameOrigin_X" value="0.0"/>
+  <xacro:property name="ForearmMassSimFrameOrigin_Y" value="0.0"/>
+  <xacro:property name="ForearmMassSimFrameOrigin_Z" value="0.0"/>
+  <xacro:property name="ForearmMassSimFrameOrientation_Roll" value="0.0"/>
+  <xacro:property name="ForearmMassSimFrameOrientation_Pitch" value="0.0"/>
+  <xacro:property name="ForearmMassSimFrameOrientation_Yaw" value="0.0"/>
   <xacro:property name="WristRollFrameOrigin_X" value="0.0"/>
   <xacro:property name="WristRollFrameOrigin_Y" value="${reflect * 0.2871}"/>

File: model/robots/common/xacro/arm/mass_parameters.xacro (robot description, xacro)
@@ -41,4 +41,12 @@
   <xacro:property name="ForearmYawLinkInertia_IYZ" value="${reflect*0.001695416}" />
   <xacro:property name="ForearmYawLinkInertia_IZZ" value="0.011365657" />
+  <xacro:property name="ForearmMassSimLinkMass" value="4.2" />
+  <xacro:property name="ForearmMassSimComPosition" value="0.015000  ${reflect*0.13} 0.019564" />
+  <xacro:property name="ForearmMassSimInertia_IXX" value="0.011755430" />
+  <xacro:property name="ForearmMassSimInertia_IXY" value="${reflect*0.001300853}" />
+  <xacro:property name="ForearmMassSimInertia_IXZ" value="-0.000727141" />
+  <xacro:property name="ForearmMassSimInertia_IYY" value="0.005071567" />
+  <xacro:property name="ForearmMassSimInertia_IYZ" value="${reflect*0.001695416}" />
+  <xacro:property name="ForearmMassSimInertia_IZZ" value="0.011365657" />
   <xacro:property name="WristRollLinkMass" value="0.14" />
   <xacro:property name="WristRollLinkComPosition" value="0 ${reflect*0} 0" />

File: model/robots/valkyrie_sim_mass_sims.xacro (robot description, xacro)
@@ -7,4 +7,4 @@
     <xacro:include filename="$(find val_description)/common/xacro/serial_numbers/valkyrie_A_serials.xacro"/>
     <xacro:include filename="$(find val_description)/common/xacro/dev_ports/valkyrie_gazebo_ports.xacro"/>
-    <xacro:include filename="$(find val_description)/model/robots/common/xacro/valkyrie_arm_mass_sims_base_hw.xacro"/>
+    <xacro:include filename="$(find val_description)/model/robots/common/xacro/valkyrie_arm_mass_sims_base_sim.xacro"/>
 </robot>

Commit message: Changed mesh of elbow link to that of elbow link and forearm mass sim combined for arm mass sim val urdf creation

File: model/robots/common/xacro/arm/arm.xacro (robot description, xacro)
@@ -152,6 +152,36 @@
     </xacro:revolute_joint_ex>
   </xacro:macro>
-    <xacro:macro name="make_lower_arm_mass_sim" params="prefix reflect lower_arm_root_link">
-    <xacro:standard_link name="${ForearmLinkName}"
+  <xacro:macro name="make_arm" params="prefix reflect arm_root_link">
+    <xacro:make_upper_arm prefix="${prefix}" reflect="${reflect}" upper_arm_root_link="${arm_root_link}" />
+    <xacro:make_lower_arm prefix="${prefix}" reflect="${reflect}" lower_arm_root_link="${ElbowPitchLinkName}" />
+  </xacro:macro>
+  <xacro:macro name="make_arm_no_hands" params="prefix reflect arm_root_link">
+    <xacro:make_upper_arm prefix="${prefix}" reflect="${reflect}" upper_arm_root_link="${arm_root_link}" />
+  </xacro:macro>
+  <xacro:macro name="make_arm_mass_sims" params="prefix reflect arm_root_link">
+    <xacro:standard_link name="${ShoulderPitchLinkName}"
+                    mass="${ShoulderPitchLinkMass}"
+                    origin_xyz="${ShoulderPitchLinkComPosition}" origin_rpy="0 0 0"
+                    ixx="${ShoulderPitchLinkInertia_IXX}" ixy="${ShoulderPitchLinkInertia_IXY}" ixz="${ShoulderPitchLinkInertia_IXZ}"
+                    iyy="${ShoulderPitchLinkInertia_IYY}" iyz="${ShoulderPitchLinkInertia_IYZ}" izz="${ShoulderPitchLinkInertia_IZZ}"
+                    visual_mesh="${mesh_root}/arms/aj1_${prefix}.dae"
+                    collision_mesh="${mesh_root}/arms/aj1_${prefix}.dae" />
+    <xacro:standard_link name="${ShoulderRollLinkName}"
+                    mass="${ShoulderRollLinkMass}"
+                    origin_xyz="${ShoulderRollLinkComPosition}"
+                    ixx="${ShoulderRollLinkInertia_IXX}" ixy="${ShoulderRollLinkInertia_IXY}" ixz="${ShoulderRollLinkInertia_IXZ}"
+                    iyy="${ShoulderRollLinkInertia_IYY}" iyz="${ShoulderRollLinkInertia_IYZ}" izz="${ShoulderRollLinkInertia_IZZ}"
+                    origin_rpy="0 0 0"
+                    visual_mesh="${mesh_root}/arms/aj2_${prefix}.dae"
+                    collision_mesh="${mesh_root}/arms/aj2_${prefix}.dae" />
+    <xacro:standard_link name="${ShoulderYawLinkName}"
+                    mass="${ShoulderYawLinkMass}"
+                    origin_xyz="${ShoulderYawLinkComPosition}"
+                    ixx="${ShoulderYawLinkInertia_IXX}" ixy="${ShoulderYawLinkInertia_IXY}" ixz="${ShoulderYawLinkInertia_IXZ}"
+                    iyy="${ShoulderYawLinkInertia_IYY}" iyz="${ShoulderYawLinkInertia_IYZ}" izz="${ShoulderYawLinkInertia_IZZ}"
+                    origin_rpy="0 0 0"
+                    visual_mesh="${mesh_root}/arms/aj3_${prefix}.dae"
+                    collision_mesh="${mesh_root}/arms/aj3_${prefix}.dae" />
+    <xacro:standard_link name="${ElbowPitchLinkName}"
                     mass="${ForearmMassSimLinkMass}"
                     origin_xyz="${ForearmMassSimComPosition}"
@@ -161,20 +191,50 @@
                     visual_mesh="${mesh_root}/arms/${prefix}_elbow_mass_sim.dae"
                     collision_mesh="${mesh_root}/arms/${prefix}_elbow_mass_sim.dae" />
-    <xacro:fixed_joint jointName="${ForearmYawJointName}"
-                          parent="${lower_arm_root_link}" child="${ForearmLinkName}"
-                          origin_xyz="${ForearmMassSimFrameOrigin_X} ${ForearmMassSimFrameOrigin_Y} ${ForearmMassSimFrameOrigin_Z}"
-                          origin_rpy="${ForearmMassSimFrameOrientation_Roll} ${ForearmMassSimFrameOrientation_Pitch} ${ForearmMassSimFrameOrientation_Yaw}">
-    </xacro:fixed_joint>
-  </xacro:macro>
-  <xacro:macro name="make_arm" params="prefix reflect arm_root_link">
-    <xacro:make_upper_arm prefix="${prefix}" reflect="${reflect}" upper_arm_root_link="${arm_root_link}" />
-    <xacro:make_lower_arm prefix="${prefix}" reflect="${reflect}" lower_arm_root_link="${ElbowPitchLinkName}" />
-  </xacro:macro>
-  <xacro:macro name="make_arm_no_hands" params="prefix reflect arm_root_link">
-    <xacro:make_upper_arm prefix="${prefix}" reflect="${reflect}" upper_arm_root_link="${arm_root_link}" />
-  </xacro:macro>
-  <xacro:macro name="make_arm_mass_sims" params="prefix reflect arm_root_link">
-    <xacro:make_upper_arm prefix="${prefix}" reflect="${reflect}" upper_arm_root_link="${arm_root_link}" />
-    <xacro:make_lower_arm_mass_sim prefix="${prefix}" reflect="${reflect}" lower_arm_root_link="${ElbowPitchLinkName}" />
+    <xacro:revolute_joint_ex jointName="${ShoulderPitchJointName}"
+                          parent="${arm_root_link}" child="${ShoulderPitchLinkName}"
+                          origin_xyz="${ShoulderPitchFrameOrigin_X} ${ShoulderPitchFrameOrigin_Y} ${ShoulderPitchFrameOrigin_Z}"
+                          origin_rpy="${ShoulderPitchFrameOrientation_Roll} ${ShoulderPitchFrameOrientation_Pitch} ${ShoulderPitchFrameOrientation_Yaw}"
+                          axis="${ShoulderPitchRotationAxis}"
+                          damping="0.1" friction="0.0">
+        <limit effort="${ShoulderPitchTorqueLimit}" lower="${ShoulderPitchPositionLimit_Lower}" upper="${ShoulderPitchPositionLimit_Upper}" velocity="${ShoulderPitchVelocityLimit}"/>
+        <controller_gains Kp="0.0" Kd="0.0" Ki="0.0"/>
+    </xacro:revolute_joint_ex>
+    <xacro:revolute_joint_ex jointName="${ShoulderRollJointName}"
+                          parent="${ShoulderPitchLinkName}" child="${ShoulderRollLinkName}"
+                          origin_xyz="${ShoulderRollFrameOrigin_X} ${ShoulderRollFrameOrigin_Y} ${ShoulderRollFrameOrigin_Z}"
+                          origin_rpy="${ShoulderRollFrameOrientation_Roll} ${ShoulderRollFrameOrientation_Pitch} ${ShoulderRollFrameOrientation_Yaw}"
+                          axis="${ShoulderRollRotationAxis}"
+                          damping="0.1" friction="0.0">
+        <xacro:if value="${(reflect+1)/2}">
+        <limit effort="${ShoulderRollTorqueLimit}" lower="${ShoulderRollPositionLimit_Lower}" upper="${ShoulderRollPositionLimit_Upper}" velocity="${ShoulderRollVelocityLimit}"/>
+        </xacro:if>
+        <xacro:if value="${(-reflect+1)/2}">
+        <limit effort="${ShoulderRollTorqueLimit}" lower="${reflect * ShoulderRollPositionLimit_Upper}" upper="${reflect * ShoulderRollPositionLimit_Lower}" velocity="${ShoulderRollVelocityLimit}"/>
+        </xacro:if>
+        <controller_gains Kp="0.0" Kd="0.0" Ki="0.0"/>
+    </xacro:revolute_joint_ex>
+    <xacro:revolute_joint_ex jointName="${ShoulderYawJointName}"
+                          parent="${ShoulderRollLinkName}" child="${ShoulderYawLinkName}"
+                          origin_xyz="${ShoulderYawFrameOrigin_X} ${ShoulderYawFrameOrigin_Y} ${ShoulderYawFrameOrigin_Z}"
+                          origin_rpy="${ShoulderYawFrameOrientation_Roll} ${ShoulderYawFrameOrientation_Pitch} ${ShoulderYawFrameOrientation_Yaw}"
+                          axis="${ShoulderYawRotationAxis}"
+                          damping="0.1" friction="0.0">
+        <limit effort="${ShoulderYawTorqueLimit}" lower="${ShoulderYawPositionLimit_Lower}" upper="${ShoulderYawPositionLimit_Upper}" velocity="${ShoulderYawVelocityLimit}"/>
+        <controller_gains Kp="0.0" Kd="0.0" Ki="0.0"/>
+    </xacro:revolute_joint_ex>
+    <xacro:revolute_joint_ex jointName="${ElbowPitchJointName}"
+                          parent="${ShoulderYawLinkName}" child="${ElbowPitchLinkName}"
+                          origin_xyz="${ElbowPitchFrameOrigin_X} ${ElbowPitchFrameOrigin_Y} ${ElbowPitchFrameOrigin_Z}"
+                          origin_rpy="${ElbowPitchFrameOrientation_Roll} ${ElbowPitchFrameOrientation_Pitch} ${ElbowPitchFrameOrientation_Yaw}"
+                          axis="${ElbowPitchRotationAxis}"
+                          damping="0.1" friction="0.0">
+        <xacro:if value="${(reflect+1)/2}">
+        <limit effort="${ElbowPitchTorqueLimit}" lower="${ElbowPitchPositionLimit_Lower}" upper="${ElbowPitchPositionLimit_Upper}" velocity="${ElbowPitchVelocityLimit}"/>
+        </xacro:if>
+        <xacro:if value="${(-reflect+1)/2}">
+        <limit effort="${ElbowPitchTorqueLimit}" lower="${reflect * ElbowPitchPositionLimit_Upper}" upper="${reflect * ElbowPitchPositionLimit_Lower}" velocity="${ElbowPitchVelocityLimit}"/>
+        </xacro:if>
+        <controller_gains Kp="0.0" Kd="0.0" Ki="0.0"/>
+    </xacro:revolute_joint_ex>
   </xacro:macro>
   <xacro:macro name="arm_transmissions_hw" params="prefix reflect">

File: model/robots/common/xacro/arm/frame_parameters.xacro (robot description, xacro)
@@ -31,10 +31,4 @@
   <xacro:property name="ForearmYawFrameOrientation_Pitch" value="0.0"/>
   <xacro:property name="ForearmYawFrameOrientation_Yaw" value="0.0"/>
-  <xacro:property name="ForearmMassSimFrameOrigin_X" value="0.0"/>
-  <xacro:property name="ForearmMassSimFrameOrigin_Y" value="0.0"/>
-  <xacro:property name="ForearmMassSimFrameOrigin_Z" value="0.0"/>
-  <xacro:property name="ForearmMassSimFrameOrientation_Roll" value="0.0"/>
-  <xacro:property name="ForearmMassSimFrameOrientation_Pitch" value="0.0"/>
-  <xacro:property name="ForearmMassSimFrameOrientation_Yaw" value="0.0"/>
   <xacro:property name="WristRollFrameOrigin_X" value="0.0"/>
   <xacro:property name="WristRollFrameOrigin_Y" value="${reflect * 0.2871}"/>

File: model/robots/common/xacro/arm/mass_parameters.xacro (robot description, xacro)
@@ -33,4 +33,12 @@
   <xacro:property name="ElbowPitchLinkInertia_IYZ" value="-0.000423865" />
   <xacro:property name="ElbowPitchLinkInertia_IZZ" value="0.003011283" />
+  <xacro:property name="ForearmMassSimLinkMass" value="6.03" />
+  <xacro:property name="ForearmMassSimComPosition" value="-0.010000  ${reflect*0.13} 0.019564" />
+  <xacro:property name="ForearmMassSimInertia_IXX" value="0.011755430" />
+  <xacro:property name="ForearmMassSimInertia_IXY" value="${reflect*0.001300853}" />
+  <xacro:property name="ForearmMassSimInertia_IXZ" value="-0.000727141" />
+  <xacro:property name="ForearmMassSimInertia_IYY" value="0.005071567" />
+  <xacro:property name="ForearmMassSimInertia_IYZ" value="${reflect*0.001695416}" />
+  <xacro:property name="ForearmMassSimInertia_IZZ" value="0.011365657" />
   <xacro:property name="ForearmYawLinkMass" value="2.476" />
   <xacro:property name="ForearmYawLinkComPosition" value="0.015000	${reflect*0.13} 0.019564" />
@@ -41,12 +49,4 @@
   <xacro:property name="ForearmYawLinkInertia_IYZ" value="${reflect*0.001695416}" />
   <xacro:property name="ForearmYawLinkInertia_IZZ" value="0.011365657" />
-  <xacro:property name="ForearmMassSimLinkMass" value="4.2" />
-  <xacro:property name="ForearmMassSimComPosition" value="0.015000  ${reflect*0.13} 0.019564" />
-  <xacro:property name="ForearmMassSimInertia_IXX" value="0.011755430" />
-  <xacro:property name="ForearmMassSimInertia_IXY" value="${reflect*0.001300853}" />
-  <xacro:property name="ForearmMassSimInertia_IXZ" value="-0.000727141" />
-  <xacro:property name="ForearmMassSimInertia_IYY" value="0.005071567" />
-  <xacro:property name="ForearmMassSimInertia_IYZ" value="${reflect*0.001695416}" />
-  <xacro:property name="ForearmMassSimInertia_IZZ" value="0.011365657" />
   <xacro:property name="WristRollLinkMass" value="0.14" />
   <xacro:property name="WristRollLinkComPosition" value="0 ${reflect*0} 0" />

Commit message: Fixed transmissions in new mass sims macro for the arm.

File: model/robots/common/xacro/arm/arm.xacro (robot description, xacro)
@@ -262,3 +262,9 @@
     <xacro:simple_position_transmission jointName="${WristPitchJointName}" actuatorName="${WristPitchActuatorSimName}" nodeName="${WristPitchActuatorSimNode}" actuatorApi="${SimApi}"/>
   </xacro:macro>
+  <xacro:macro name="arm_transmissions_sim_no_hands" params="prefix">
+    <xacro:simple_transmission jointName="${ShoulderPitchJointName}" actuatorName="${ShoulderPitchActuatorName}" nodeName="${ShoulderPitchNode}" actuatorApi="${SimApi}"/>
+    <xacro:simple_transmission jointName="${ShoulderRollJointName}" actuatorName="${ShoulderRollActuatorName}" nodeName="${ShoulderRollNode}" actuatorApi="${SimApi}"/>
+    <xacro:simple_transmission jointName="${ShoulderYawJointName}" actuatorName="${ShoulderYawActuatorName}" nodeName="${ShoulderYawNode}" actuatorApi="${SimApi}"/>
+    <xacro:simple_transmission jointName="${ElbowPitchJointName}" actuatorName="${ElbowPitchActuatorName}" nodeName="${ElbowPitchNode}" actuatorApi="${SimApi}"/>
+  </xacro:macro>
 </robot>

File: model/robots/common/xacro/valkyrie_arm_mass_sims_base_sim.xacro (robot description, xacro)
@@ -20,6 +20,6 @@
     <xacro:leg_transmissions_sim prefix="left"/>
     <xacro:leg_transmissions_sim prefix="right"/>
-    <xacro:arm_transmissions_sim prefix="left"/>
-    <xacro:arm_transmissions_sim prefix="right"/>
+    <xacro:arm_transmissions_sim_no_hands prefix="left"/>
+    <xacro:arm_transmissions_sim_no_hands prefix="right"/>
     <xacro:neck_transmissions_sim />
 </robot>
