Commit message: added virtual link for six axis force torque sensors

File: model/robots/common/xacro/leg/leg.xacro (robot description, xacro)
@@ -143,5 +143,4 @@
     <xacro:ati_force_torque_sensor sensorName="${prefix}FootSixAxis"
                         parentLink="${AnkleRollLinkName}"
-                        joint_to_attach_sensor_to="${AnkleRollJointName}"
                         origin_xyz="0.0215646 0.0 -0.051054"
                         origin_rpy="3.14 0.0 0.0"

File: model/robots/common/xacro/sensors/ati_force_torque.xacro (robot description, xacro)
@@ -1,8 +1,15 @@
 <?xml version="1.0" ?>
 <robot xmlns:xacro="http://www.ros.org/wiki/xacro" name="ati_force_torque_sensor">
-  <xacro:macro name="ati_force_torque_sensor" params="sensorName parentLink joint_to_attach_sensor_to origin_xyz origin_rpy sensor_number sensor_node sensor_api">
-    <gazebo reference="${joint_to_attach_sensor_to}">
+  <xacro:macro name="ati_force_torque_sensor" params="sensorName parentLink origin_xyz origin_rpy sensor_number sensor_node sensor_api">
+    <xacro:massless_virtual_link name="${sensorName}_Frame"
+                    origin_rpy="0 0 0"
+                    origin_xyz="0 0 0"/>
+    <xacro:fixed_joint jointName="${sensorName}_Offset"
+                       parent="${parentLink}" child="${sensorName}_Frame"
+                       origin_rpy="${origin_rpy}"
+                       origin_xyz="${origin_xyz}"/>
+    <gazebo reference="${sensorName}_Frame">
       <sensor name="${sensorName}" type="force_torque">
-        <pose>${origin_xyz} ${origin_rpy}</pose>
+        <pose>0 0 0 0 0 0 </pose>
         <sensor_number id="${sensor_number}" />
         <node id="${sensor_node}" />
