Commit message: added firmware to instances

File: instance/instances/robots/forearm_testbench_left.xacro (robot description, xacro)
@@ -9,5 +9,5 @@
     </Channels>
     <Mechanisms>
-    <xacro:simple_mechanism name="testbench_actuator" serial_number="${forearm_yaw_serial_number}" node="${testbench_node}"/>
+    <xacro:simple_mechanism name="testbench_actuator" serial_number="${forearm_yaw_serial_number}" node="${testbench_node}" processor_firmware="" fpga_firmware=""/>
     <xacro:forearm mechanism_name="${prefix}Forearm" serial_number="${forearm_serial_number}" athena1_node="${Athena1Node}" athena2_node="${Athena2Node}" />
 	</Mechanisms>

File: instance/instances/robots/forearm_testbench_right.xacro (robot description, xacro)
@@ -9,5 +9,5 @@
     </Channels>
     <Mechanisms>
-    <xacro:simple_mechanism name="testbench_actuator" serial_number="${forearm_yaw_serial_number}" node="${testbench_node}"/>
+    <xacro:simple_mechanism name="testbench_actuator" serial_number="${forearm_yaw_serial_number}" node="${testbench_node}" processor_firmware="" fpga_firmware=""/>
     <xacro:forearm mechanism_name="${prefix}Forearm" serial_number="${forearm_serial_number}" athena1_node="${Athena1Node}" athena2_node="${Athena2Node}" />
 	</Mechanisms>

File: instance/instances/robots/xacro/common/valkyrie_full_template.xacro (robot description, xacro)
@@ -9,4 +9,5 @@
 	<RobotInstance id="${instance}" />
 	<xacro:all_channels/>
+	<xacro:firmware_base_url/>
 	<Mechanisms>
 		<xacro:leg prefix="left" j1_serial_number="${leftLegJ1SerialNumber}" j2_serial_number="${leftLegJ2SerialNumber}" j3_serial_number="${leftLegJ3SerialNumber}" j4_serial_number="${leftLegJ4SerialNumber}" ankle_left_actuator_serial="${leftAnkleLeftActuatorSerialNumber}" ankle_right_actuator_serial="${leftAnkleRightActuatorSerialNumber}"/>

File: instance/instances/robots/xacro/limbs/arm.xacro (robot description, xacro)
@@ -2,10 +2,11 @@
     <xacro:include filename="$(find val_description)/instance/instances/robots/xacro/mechanisms/mechanisms.xacro"/>
     <xacro:include filename="$(find val_description)/common/xacro/joint_names/valkyrie_joint_names.xacro"/>
+    <xacro:include filename="$(find val_description)/common/xacro/firmware/valkyrie_firmware.xacro"/>
     <xacro:macro name="arm" params="prefix j1_serial_number j2_serial_number j3_serial_number j4_serial_number j5_serial_number forearm_serial_number" >
-    	<xacro:simple_mechanism name="${ShoulderPitchJointName}" serial_number="${j1_serial_number}" node="${ShoulderPitchNode}"/>
-    	<xacro:simple_mechanism name="${ShoulderRollJointName}" serial_number="${j2_serial_number}" node="${ShoulderRollNode}"/>
-    	<xacro:simple_mechanism name="${ShoulderYawJointName}" serial_number="${j3_serial_number}" node="${ShoulderYawNode}"/>
-    	<xacro:simple_mechanism name="${ElbowPitchJointName}" serial_number="${j4_serial_number}" node="${ElbowPitchNode}"/>
-    	<xacro:simple_mechanism name="${ForearmYawJointName}" serial_number="${j5_serial_number}" node="${ForearmYawNode}"/>
+    	<xacro:simple_mechanism name="${ShoulderPitchJointName}" serial_number="${j1_serial_number}" node="${ShoulderPitchNode}" processor_firmware="${TurboProcRotaryFirmwareURL}" fpga_firmware="${TurboFPGAFirmwareURL}"/>
+    	<xacro:simple_mechanism name="${ShoulderRollJointName}" serial_number="${j2_serial_number}" node="${ShoulderRollNode}" processor_firmware="${TurboProcRotaryFirmwareURL}" fpga_firmware="${TurboFPGAFirmwareURL}"/>
+    	<xacro:simple_mechanism name="${ShoulderYawJointName}" serial_number="${j3_serial_number}" node="${ShoulderYawNode}" processor_firmware="${TurboProcRotaryFirmwareURL}" fpga_firmware="${TurboFPGAFirmwareURL}"/>
+    	<xacro:simple_mechanism name="${ElbowPitchJointName}" serial_number="${j4_serial_number}" node="${ElbowPitchNode}" processor_firmware="${TurboProcRotaryFirmwareURL}" fpga_firmware="${TurboFPGAFirmwareURL}"/>
+    	<xacro:simple_mechanism name="${ForearmYawJointName}" serial_number="${j5_serial_number}" node="${ForearmYawNode}" processor_firmware="" fpga_firmware=""/>
         <xacro:forearm mechanism_name="${prefix}Forearm" serial_number="${forearm_serial_number}" athena1_node="${Athena1Node}" athena2_node="${Athena2Node}" />
     </xacro:macro>

File: instance/instances/robots/xacro/limbs/leg.xacro (robot description, xacro)
@@ -3,9 +3,9 @@
     <xacro:include filename="$(find val_description)/common/xacro/joint_names/valkyrie_joint_names.xacro"/>
     <xacro:macro name="leg" params="prefix j1_serial_number j2_serial_number j3_serial_number j4_serial_number ankle_left_actuator_serial ankle_right_actuator_serial" >
-    	<xacro:simple_mechanism name="${HipYawJointName}" serial_number="${j1_serial_number}" node="${HipYawNode}"/>
-    	<xacro:simple_mechanism name="${HipRollJointName}" serial_number="${j2_serial_number}" node="${HipRollNode}"/>
-    	<xacro:simple_mechanism name="${HipPitchJointName}" serial_number="${j3_serial_number}" node="${HipPitchNode}"/>
-    	<xacro:simple_mechanism name="${KneePitchJointName}" serial_number="${j4_serial_number}" node="${KneePitchNode}"/>
-    	<xacro:two_active_joint_mechanism mechanism_name="${prefix}Ankle" actuator0_name="${AnkleLeftActuatorName}" actuator1_name="${AnkleRightActuatorName}" joint0_name="${AnklePitchJointName}" joint1_name="${AnkleRollJointName}" actuator0_serial="${ankle_left_actuator_serial}" actuator1_serial="${ankle_right_actuator_serial}" actuator0_node="${AnkleLeftActuatorNode}" actuator1_node="${AnkleRightActuatorNode}" />
+    	<xacro:simple_mechanism name="${HipYawJointName}" serial_number="${j1_serial_number}" node="${HipYawNode}" processor_firmware="${TurboProcRotaryFirmwareURL}" fpga_firmware="${TurboFPGAFirmwareURL}"/>
+    	<xacro:simple_mechanism name="${HipRollJointName}" serial_number="${j2_serial_number}" node="${HipRollNode}" processor_firmware="${TurboProcRotaryFirmwareURL}" fpga_firmware="${TurboFPGAFirmwareURL}"/>
+    	<xacro:simple_mechanism name="${HipPitchJointName}" serial_number="${j3_serial_number}" node="${HipPitchNode}" processor_firmware="${TurboProcRotaryFirmwareURL}" fpga_firmware="${TurboFPGAFirmwareURL}"/>
+    	<xacro:simple_mechanism name="${KneePitchJointName}" serial_number="${j4_serial_number}" node="${KneePitchNode}" processor_firmware="${TurboProcRotaryFirmwareURL}" fpga_firmware="${TurboFPGAFirmwareURL}"/>
+    	<xacro:two_active_joint_mechanism mechanism_name="${prefix}Ankle" actuator0_name="${AnkleLeftActuatorName}" actuator1_name="${AnkleRightActuatorName}" joint0_name="${AnklePitchJointName}" joint1_name="${AnkleRollJointName}" actuator0_serial="${ankle_left_actuator_serial}" actuator1_serial="${ankle_right_actuator_serial}" actuator0_node="${AnkleLeftActuatorNode}" actuator1_node="${AnkleRightActuatorNode}" processor_firmware0="${TurboProcLinearFirmwareURL}" fpga_firmware0="${TurboFPGAFirmwareURL}"/>
     </xacro:macro>
 </robot>

File: instance/instances/robots/xacro/limbs/neck.xacro (robot description, xacro)
@@ -3,7 +3,7 @@
     <xacro:include filename="$(find val_description)/common/xacro/joint_names/valkyrie_joint_names.xacro"/>
     <xacro:macro name="neck" params="j1_serial_number j2_serial_number j3_serial_number" >
-    	<xacro:simple_mechanism name="${LowerNeckPitchJointName}" serial_number="${j1_serial_number}" node="${LowerNeckPitchNode}"/>
-    	<xacro:simple_mechanism name="${NeckYawJointName}" serial_number="${j2_serial_number}" node="${NeckYawNode}"/>
-    	<xacro:simple_mechanism name="${UpperNeckPitchJointName}" serial_number="${j3_serial_number}" node="${UpperNeckPitchNode}"/>
+    	<xacro:simple_mechanism name="${LowerNeckPitchJointName}" serial_number="${j1_serial_number}" node="${LowerNeckPitchNode}" processor_firmware="" fpga_firmware=""/>
+    	<xacro:simple_mechanism name="${NeckYawJointName}" serial_number="${j2_serial_number}" node="${NeckYawNode}" processor_firmware="" fpga_firmware=""/>
+    	<xacro:simple_mechanism name="${UpperNeckPitchJointName}" serial_number="${j3_serial_number}" node="${UpperNeckPitchNode}" processor_firmware="" fpga_firmware=""/>
     </xacro:macro>
 </robot>

File: instance/instances/robots/xacro/limbs/waist.xacro (robot description, xacro)
@@ -4,6 +4,6 @@
     <xacro:include filename="$(find val_description)/common/xacro/actuator_names/valkyrie_actuator_names.xacro"/>
     <xacro:macro name="waist" params="j1_serial_number waist_left_actuator_serial waist_right_actuator_serial" >
-    	<xacro:simple_mechanism name="${TorsoYawJointName}" serial_number="${j1_serial_number}" node="${TrunkYawNode}"/>
-    	<xacro:two_active_joint_mechanism mechanism_name="waist" actuator0_name="${WaistLeftActuatorName}" actuator1_name="${WaistRightActuatorName}" joint0_name="${TorsoPitchJointName}" joint1_name="${TorsoRollJointName}" actuator0_serial="${waist_left_actuator_serial}" actuator1_serial="${waist_right_actuator_serial}" actuator0_node="${WaistLeftActuatorNode}" actuator1_node="${WaistRightActuatorNode}" />
+    	<xacro:simple_mechanism name="${TorsoYawJointName}" serial_number="${j1_serial_number}" node="${TrunkYawNode}" processor_firmware="${TurboProcRotaryFirmwareURL}" fpga_firmware="${TurboFPGAFirmwareURL}"/>
+    	<xacro:two_active_joint_mechanism mechanism_name="waist" actuator0_name="${WaistLeftActuatorName}" actuator1_name="${WaistRightActuatorName}" joint0_name="${TorsoPitchJointName}" joint1_name="${TorsoRollJointName}" actuator0_serial="${waist_left_actuator_serial}" actuator1_serial="${waist_right_actuator_serial}" actuator0_node="${WaistLeftActuatorNode}" actuator1_node="${WaistRightActuatorNode}" processor_firmware0="${TurboProcLinearFirmwareURL}" fpga_firmware0="${TurboFPGAFirmwareURL}"/>/>
     </xacro:macro>
 </robot>

File: instance/instances/robots/xacro/mechanisms/mechanisms.xacro (robot description, xacro)
@@ -1,7 +1,9 @@
 <robot xmlns:xacro="http://ros.org/wiki/xacro" name="actuators">
-  <xacro:macro name="simple_mechanism" params="name serial_number node">
+  <xacro:macro name="simple_mechanism" params="name serial_number node processor_firmware fpga_firmware">
   	<Mechanism id="${name}" type="simple">
   		<SerialNumber id="${serial_number}" />
   		<Node id="${node}" />
+  		<Processor_Firmware id="${processor_firmware}" />
+  		<Fpga_Firmware id="${fpga_firmware}" />
 	</Mechanism>
 </xacro:macro>
@@ -10,16 +12,18 @@
 	</Joint>
 </xacro:macro>
-<xacro:macro name="actuator" params="name serial_number node" >
+<xacro:macro name="actuator" params="name serial_number node processor_firmware fpga_firmware" >
 	<Actuator id="${name}">
 		<SerialNumber id="${serial_number}" />
 		<Node id="${node}" />
+		<Processor_Firmware id="${processor_firmware}" />
+		<Fpga_Firmware id="${fpga_firmware}" />
 	</Actuator>
 </xacro:macro>
-<xacro:macro name="two_active_joint_mechanism" params="mechanism_name actuator0_name actuator1_name joint0_name joint1_name actuator0_serial actuator0_node actuator1_serial actuator1_node " >
+<xacro:macro name="two_active_joint_mechanism" params="mechanism_name actuator0_name actuator1_name joint0_name joint1_name actuator0_serial actuator0_node actuator1_serial actuator1_node processor_firmware0 fpga_firmware0" >
 	<Mechanism id="${mechanism_name}" type="complex">
 		<xacro:joint name="${joint0_name}" type="active"/>
 		<xacro:joint name="${joint1_name}" type="active"/>
-		<xacro:actuator name="${actuator0_name}" serial_number="${actuator0_serial}" node="${actuator0_node}" />
-		<xacro:actuator name="${actuator1_name}" serial_number="${actuator1_serial}" node="${actuator1_node}" />
+		<xacro:actuator name="${actuator0_name}" serial_number="${actuator0_serial}" node="${actuator0_node}" processor_firmware="${processor_firmware0}" fpga_firmware="${fpga_firmware0}"/>
+		<xacro:actuator name="${actuator1_name}" serial_number="${actuator1_serial}" node="${actuator1_node}" processor_firmware="${processor_firmware0}" fpga_firmware="${fpga_firmware0}"/>
 	</Mechanism>
 </xacro:macro>
