Commit message: calibration and torque control fixes for unit A

File: common/xacro/dev_ports/valkyrie_A_ports.xacro (robot description, xacro)
@@ -1,5 +1,5 @@
 <robot xmlns:xacro="http://ros.org/wiki/xacro" name="valkyrie_A_ports">
 	<xacro:property name="pelvis_middle_imu_port" value="/dev/ttyACM0" />
-	<xacro:property name="pelvis_rear_imu_port" value="/dev/ttyACM0" />
-	<xacro:property name="torso_left_imu_port" value="/dev/ttyACM0" />
+	<xacro:property name="pelvis_rear_imu_port" value="/dev/serial/by-id/usb-Lord_Microstrain_Lord_Inertial_Sensor_0000__6233.47095-if00" />
+	<xacro:property name="torso_left_imu_port" value="/dev/serial/by-id/usb-Lord_Microstrain_Lord_Inertial_Sensor_0000__6233.47090-if00" />
 </robot>

Commit message: switched imu and torque offset for linear in torso

File: common/xacro/dev_ports/valkyrie_A_ports.xacro (robot description, xacro)
@@ -1,5 +1,5 @@
 <robot xmlns:xacro="http://ros.org/wiki/xacro" name="valkyrie_A_ports">
 	<xacro:property name="pelvis_middle_imu_port" value="/dev/ttyACM0" />
-	<xacro:property name="pelvis_rear_imu_port" value="/dev/serial/by-id/usb-Lord_Microstrain_Lord_Inertial_Sensor_0000__6233.47095-if00" />
+	<xacro:property name="pelvis_rear_imu_port" value="/dev/serial/by-id/usb-Lord_Microstrain_Lord_Inertial_Sensor_0000__6233.47092-if00" />
 	<xacro:property name="torso_left_imu_port" value="/dev/serial/by-id/usb-Lord_Microstrain_Lord_Inertial_Sensor_0000__6233.47090-if00" />
 </robot>

Commit message: changed imu back

File: common/xacro/dev_ports/valkyrie_A_ports.xacro (robot description, xacro)
@@ -1,5 +1,5 @@
 <robot xmlns:xacro="http://ros.org/wiki/xacro" name="valkyrie_A_ports">
 	<xacro:property name="pelvis_middle_imu_port" value="/dev/ttyACM0" />
-	<xacro:property name="pelvis_rear_imu_port" value="/dev/serial/by-id/usb-Lord_Microstrain_Lord_Inertial_Sensor_0000__6233.47092-if00" />
+	<xacro:property name="pelvis_rear_imu_port" value="/dev/serial/by-id/usb-Lord_Microstrain_Lord_Inertial_Sensor_0000__6233.47095-if00" />
 	<xacro:property name="torso_left_imu_port" value="/dev/serial/by-id/usb-Lord_Microstrain_Lord_Inertial_Sensor_0000__6233.47090-if00" />
 </robot>
