Commit message: added joint specific firmware in xacros

File: common/xacro/firmware/valkyrie_firmware.xacro (robot description, xacro)
@@ -1,6 +1,8 @@
 <?xml version="1.0" ?>
 <robot name="valkyrie_firmware_locations" xmlns:xacro="http://www.ros.org/wiki/xacro">
-    <xacro:property name="ProcFirmwareBaseURL" value="http://flexo.jsc.nasa.gov/bamboo/browse/DRCE-TURBOPROC/latest/artifact/shared/"/>
-    <xacro:property name="FPGAFirmwareBaseURL" value="NA"/>
+    <xacro:property name="PublicProcFirmwareBaseURL" value="http://linkthatdoesnotresolve.com"/>
+    <xacro:property name="PrivateProcFirmwareBaseURL" value="http://flexo.jsc.nasa.gov/bamboo/browse/DRCE-TURBOPROC/latest/artifact/shared/"/>
+    <xacro:property name="PublicFPGAFirmwareBaseURL" value="NA"/>
+    <xacro:property name="PrivateFPGAFirmwareBaseURL" value="NA"/>
     <xacro:property name="TurboProcRotaryFirmwareExtension" value="Rotary-Binary-for-Bootloader/turbo_bootloader.bin"/>
     <xacro:property name="TurboProcLinearFirmwareExtension" value="Linear-Binary-for-Bootloader/turbo_bootloader.bin"/>
@@ -10,9 +12,49 @@
     <xacro:macro name="firmware_base_url" >
         <TurbodriverProcessorFirmware>
-            <ProcFirmwareBaseURL id="${ProcFirmwareBaseURL}"/>
+            <PublicProcFirmwareBaseURL id="${PublicProcFirmwareBaseURL}"/>
+            <PrivateProcFirmwareBaseURL id="${PrivateProcFirmwareBaseURL}"/>
         </TurbodriverProcessorFirmware>
         <TurbodriverFPGAFirmware>
-            <FPGAFirmwareBaseURL id="${FPGAFirmwareBaseURL}"/>
+            <PublicFPGAFirmwareBaseURL id="${PublicFPGAFirmwareBaseURL}"/>
+            <PrivateFPGAFirmwareBaseURL id="${PrivateFPGAFirmwareBaseURL}"/>
         </TurbodriverFPGAFirmware>
     </xacro:macro>
+    <xacro:property name="HipYawProcFirmware" value="${TurboProcRotaryFirmwareURL}" />
+    <xacro:property name="HipYawFPGAFirmware" value="" />
+    <xacro:property name="HipRollProcFirmware" value="${TurboProcRotaryFirmwareURL}" />
+    <xacro:property name="HipRollFPGAFirmware" value="" />
+    <xacro:property name="HipPitchProcFirmware" value="${TurboProcRotaryFirmwareURL}" />
+    <xacro:property name="HipPitchFPGAFirmware" value="" />
+    <xacro:property name="KneePitchProcFirmware" value="${TurboProcRotaryFirmwareURL}" />
+    <xacro:property name="KneePitchFPGAFirmware" value="" />
+    <xacro:property name="AnkleLeftActuatorProcFirmware" value="${TurboProcLinearFirmwareURL}" />
+    <xacro:property name="AnkleLeftActuatorFPGAFirmware" value="" />
+    <xacro:property name="AnkleRightActuatorProcFirmware" value="${TurboProcLinearFirmwareURL}" />
+    <xacro:property name="AnkleRightActuatorFPGAFirmware" value="" />
+    <xacro:property name="ShoulderPitchProcFirmware" value="${TurboProcRotaryFirmwareURL}" />
+    <xacro:property name="ShoulderPitchFPGAFirmware" value="" />
+    <xacro:property name="ShoulderRollProcFirmware" value="${TurboProcRotaryFirmwareURL}" />
+    <xacro:property name="ShoulderRollFPGAFirmware" value="" />
+    <xacro:property name="ShoulderYawProcFirmware" value="${TurboProcRotaryFirmwareURL}" />
+    <xacro:property name="ShoulderYawFPGAFirmware" value="" />
+    <xacro:property name="ElbowPitchProcFirmware" value="${TurboProcRotaryFirmwareURL}" />
+    <xacro:property name="ElbowPitchFPGAFirmware" value="" />
+    <xacro:property name="ForearmYawProcFirmware" value="" />
+    <xacro:property name="ForearmYawFPGAFirmware" value="" />
+    <xacro:property name="LowerNeckPitchProcessorFirmware" value="" />
+    <xacro:property name="LowerNeckPitchFPGAFirmware" value="" />
+    <xacro:property name="NeckYawProcessorFirmware" value="" />
+    <xacro:property name="NeckYawFPGAFirmware" value="" />
+    <xacro:property name="UpperNeckPitchProcessorFirmware" value="" />
+    <xacro:property name="UpperNeckPitchFPGAFirmware" value="" />
+    <xacro:property name="TrunkYawProcessorFirmware" value="${TurboProcRotaryFirmwareURL}" />
+    <xacro:property name="TrunkYawFPGAFirmware" value="" />
+    <xacro:property name="WaistRightActuatorProcessorFirmware" value="${TurboProcLinearFirmwareURL}" />
+    <xacro:property name="WaistRightActuatorFPGAFirmware" value="" />
+    <xacro:property name="WaistLeftActuatorProcessorFirmware" value="${TurboProcLinearFirmwareURL}" />
+    <xacro:property name="WaistLeftActuatorFPGAFirmware" value="" />
+    <xacro:property name="leftForearmProcessorFirmware" value=""/>
+    <xacro:property name="leftForearmFPGAFirmware" value=""/>
+    <xacro:property name="rightForearmProcessorFirmware" value=""/>
+    <xacro:property name="rightForearmFPGAFirmware" value=""/>
 </robot>

File: instance/instances/robots/xacro/limbs/arm.xacro (robot description, xacro)
@@ -4,9 +4,9 @@
     <xacro:include filename="$(find val_description)/common/xacro/firmware/valkyrie_firmware.xacro"/>
     <xacro:macro name="arm" params="prefix j1_serial_number j2_serial_number j3_serial_number j4_serial_number j5_serial_number forearm_serial_number" >
-    	<xacro:simple_mechanism name="${ShoulderPitchJointName}" serial_number="${j1_serial_number}" node="${ShoulderPitchNode}" processor_firmware="${TurboProcRotaryFirmwareURL}" fpga_firmware="${TurboFPGAFirmwareURL}"/>
-    	<xacro:simple_mechanism name="${ShoulderRollJointName}" serial_number="${j2_serial_number}" node="${ShoulderRollNode}" processor_firmware="${TurboProcRotaryFirmwareURL}" fpga_firmware="${TurboFPGAFirmwareURL}"/>
-    	<xacro:simple_mechanism name="${ShoulderYawJointName}" serial_number="${j3_serial_number}" node="${ShoulderYawNode}" processor_firmware="${TurboProcRotaryFirmwareURL}" fpga_firmware="${TurboFPGAFirmwareURL}"/>
-    	<xacro:simple_mechanism name="${ElbowPitchJointName}" serial_number="${j4_serial_number}" node="${ElbowPitchNode}" processor_firmware="${TurboProcRotaryFirmwareURL}" fpga_firmware="${TurboFPGAFirmwareURL}"/>
-    	<xacro:simple_mechanism name="${ForearmYawJointName}" serial_number="${j5_serial_number}" node="${ForearmYawNode}" processor_firmware="" fpga_firmware=""/>
+    	<xacro:simple_mechanism name="${ShoulderPitchJointName}" serial_number="${j1_serial_number}" node="${ShoulderPitchNode}" processor_firmware="${ShoulderPitchProcFirmware}" fpga_firmware="${ShoulderPitchFPGAFirmware}"/>
+    	<xacro:simple_mechanism name="${ShoulderRollJointName}" serial_number="${j2_serial_number}" node="${ShoulderRollNode}" processor_firmware="${ShoulderRollProcFirmware}" fpga_firmware="${ShoulderRollFPGAFirmware}"/>
+    	<xacro:simple_mechanism name="${ShoulderYawJointName}" serial_number="${j3_serial_number}" node="${ShoulderYawNode}" processor_firmware="${ShoulderYawProcFirmware}" fpga_firmware="${ShoulderYawFPGAFirmware}"/>
+    	<xacro:simple_mechanism name="${ElbowPitchJointName}" serial_number="${j4_serial_number}" node="${ElbowPitchNode}" processor_firmware="${ElbowPitchProcFirmware}" fpga_firmware="${ElbowPitchFPGAFirmware}"/>
+    	<xacro:simple_mechanism name="${ForearmYawJointName}" serial_number="${j5_serial_number}" node="${ForearmYawNode}" processor_firmware="${ForearmYawProcFirmware}" fpga_firmware="${ForearmYawFPGAFirmware}"/>
         <xacro:forearm mechanism_name="${prefix}Forearm" serial_number="${forearm_serial_number}" athena1_node="${Athena1Node}" athena2_node="${Athena2Node}" />
     </xacro:macro>

File: instance/instances/robots/xacro/limbs/leg.xacro (robot description, xacro)
@@ -3,9 +3,9 @@
     <xacro:include filename="$(find val_description)/common/xacro/joint_names/valkyrie_joint_names.xacro"/>
     <xacro:macro name="leg" params="prefix j1_serial_number j2_serial_number j3_serial_number j4_serial_number ankle_left_actuator_serial ankle_right_actuator_serial" >
-    	<xacro:simple_mechanism name="${HipYawJointName}" serial_number="${j1_serial_number}" node="${HipYawNode}" processor_firmware="${TurboProcRotaryFirmwareURL}" fpga_firmware="${TurboFPGAFirmwareURL}"/>
-    	<xacro:simple_mechanism name="${HipRollJointName}" serial_number="${j2_serial_number}" node="${HipRollNode}" processor_firmware="${TurboProcRotaryFirmwareURL}" fpga_firmware="${TurboFPGAFirmwareURL}"/>
-    	<xacro:simple_mechanism name="${HipPitchJointName}" serial_number="${j3_serial_number}" node="${HipPitchNode}" processor_firmware="${TurboProcRotaryFirmwareURL}" fpga_firmware="${TurboFPGAFirmwareURL}"/>
-    	<xacro:simple_mechanism name="${KneePitchJointName}" serial_number="${j4_serial_number}" node="${KneePitchNode}" processor_firmware="${TurboProcRotaryFirmwareURL}" fpga_firmware="${TurboFPGAFirmwareURL}"/>
-    	<xacro:two_active_joint_mechanism mechanism_name="${prefix}Ankle" actuator0_name="${AnkleLeftActuatorName}" actuator1_name="${AnkleRightActuatorName}" joint0_name="${AnklePitchJointName}" joint1_name="${AnkleRollJointName}" actuator0_serial="${ankle_left_actuator_serial}" actuator1_serial="${ankle_right_actuator_serial}" actuator0_node="${AnkleLeftActuatorNode}" actuator1_node="${AnkleRightActuatorNode}" processor_firmware0="${TurboProcLinearFirmwareURL}" fpga_firmware0="${TurboFPGAFirmwareURL}"/>
+    	<xacro:simple_mechanism name="${HipYawJointName}" serial_number="${j1_serial_number}" node="${HipYawNode}" processor_firmware="${HipYawProcFirmware}" fpga_firmware="${HipYawFPGAFirmware}"/>
+    	<xacro:simple_mechanism name="${HipRollJointName}" serial_number="${j2_serial_number}" node="${HipRollNode}" processor_firmware="${HipRollProcFirmware}" fpga_firmware="${HipRollFPGAFirmware}"/>
+    	<xacro:simple_mechanism name="${HipPitchJointName}" serial_number="${j3_serial_number}" node="${HipPitchNode}" processor_firmware="${HipPitchProcFirmware}" fpga_firmware="${HipPitchFPGAFirmware}"/>
+    	<xacro:simple_mechanism name="${KneePitchJointName}" serial_number="${j4_serial_number}" node="${KneePitchNode}" processor_firmware="${KneePitchProcFirmware}" fpga_firmware="${KneePitchFPGAFirmware}"/>
+    	<xacro:two_active_joint_mechanism mechanism_name="${prefix}Ankle" actuator0_name="${AnkleLeftActuatorName}" actuator1_name="${AnkleRightActuatorName}" joint0_name="${AnklePitchJointName}" joint1_name="${AnkleRollJointName}" actuator0_serial="${ankle_left_actuator_serial}" actuator1_serial="${ankle_right_actuator_serial}" actuator0_node="${AnkleLeftActuatorNode}" actuator1_node="${AnkleRightActuatorNode}" processor_firmware0="${AnkleLeftActuatorProcFirmware}" fpga_firmware0="${AnkleLeftActuatorFPGAFirmware}" processor_firmware1="${AnkleRightActuatorProcFirmware}" fpga_firmware1="${AnkleRightActuatorFPGAFirmware}"/>
     </xacro:macro>
 </robot>

File: instance/instances/robots/xacro/limbs/neck.xacro (robot description, xacro)
@@ -3,7 +3,7 @@
     <xacro:include filename="$(find val_description)/common/xacro/joint_names/valkyrie_joint_names.xacro"/>
     <xacro:macro name="neck" params="j1_serial_number j2_serial_number j3_serial_number" >
-    	<xacro:simple_mechanism name="${LowerNeckPitchJointName}" serial_number="${j1_serial_number}" node="${LowerNeckPitchNode}" processor_firmware="" fpga_firmware=""/>
-    	<xacro:simple_mechanism name="${NeckYawJointName}" serial_number="${j2_serial_number}" node="${NeckYawNode}" processor_firmware="" fpga_firmware=""/>
-    	<xacro:simple_mechanism name="${UpperNeckPitchJointName}" serial_number="${j3_serial_number}" node="${UpperNeckPitchNode}" processor_firmware="" fpga_firmware=""/>
+    	<xacro:simple_mechanism name="${LowerNeckPitchJointName}" serial_number="${j1_serial_number}" node="${LowerNeckPitchNode}" processor_firmware="${LowerNeckPitchProcessorFirmware}" fpga_firmware="${LowerNeckPitchFPGAFirmware"/>
+    	<xacro:simple_mechanism name="${NeckYawJointName}" serial_number="${j2_serial_number}" node="${NeckYawNode}" processor_firmware="${NeckYawProcessorFirmware}" fpga_firmware="${NeckYawFPGAFirmware}"/>
+    	<xacro:simple_mechanism name="${UpperNeckPitchJointName}" serial_number="${j3_serial_number}" node="${UpperNeckPitchNode}" processor_firmware="${UpperNeckPitchProcessorFirmware}" fpga_firmware="${UpperNeckPitchFPGAFirmware}"/>
     </xacro:macro>
 </robot>

File: instance/instances/robots/xacro/limbs/waist.xacro (robot description, xacro)
@@ -4,6 +4,6 @@
     <xacro:include filename="$(find val_description)/common/xacro/actuator_names/valkyrie_actuator_names.xacro"/>
     <xacro:macro name="waist" params="j1_serial_number waist_left_actuator_serial waist_right_actuator_serial" >
-    	<xacro:simple_mechanism name="${TorsoYawJointName}" serial_number="${j1_serial_number}" node="${TrunkYawNode}" processor_firmware="${TurboProcRotaryFirmwareURL}" fpga_firmware="${TurboFPGAFirmwareURL}"/>
-    	<xacro:two_active_joint_mechanism mechanism_name="waist" actuator0_name="${WaistLeftActuatorName}" actuator1_name="${WaistRightActuatorName}" joint0_name="${TorsoPitchJointName}" joint1_name="${TorsoRollJointName}" actuator0_serial="${waist_left_actuator_serial}" actuator1_serial="${waist_right_actuator_serial}" actuator0_node="${WaistLeftActuatorNode}" actuator1_node="${WaistRightActuatorNode}" processor_firmware0="${TurboProcLinearFirmwareURL}" fpga_firmware0="${TurboFPGAFirmwareURL}"/>/>
+    	<xacro:simple_mechanism name="${TorsoYawJointName}" serial_number="${j1_serial_number}" node="${TrunkYawNode}" processor_firmware="${TrunkYawProcessorFirmware}" fpga_firmware="${TrunkYawFPGAFirmware}"/>
+    	<xacro:two_active_joint_mechanism mechanism_name="waist" actuator0_name="${WaistLeftActuatorName}" actuator1_name="${WaistRightActuatorName}" joint0_name="${TorsoPitchJointName}" joint1_name="${TorsoRollJointName}" actuator0_serial="${waist_left_actuator_serial}" actuator1_serial="${waist_right_actuator_serial}" actuator0_node="${WaistLeftActuatorNode}" actuator1_node="${WaistRightActuatorNode}" processor_firmware0="${WaistLeftActuatorProcessorFirmware}" fpga_firmware0="${WaistLeftActuatorFPGAFirmware}" processor_firmware1="${WaistRightActuatorProcessorFirmware}" fpga_firmware1="${WaistRightActuatorFPGAFirmware}"/>/>
     </xacro:macro>
 </robot>

File: instance/instances/robots/xacro/mechanisms/mechanisms.xacro (robot description, xacro)
@@ -20,10 +20,10 @@
 	</Actuator>
 </xacro:macro>
-<xacro:macro name="two_active_joint_mechanism" params="mechanism_name actuator0_name actuator1_name joint0_name joint1_name actuator0_serial actuator0_node actuator1_serial actuator1_node processor_firmware0 fpga_firmware0" >
+<xacro:macro name="two_active_joint_mechanism" params="mechanism_name actuator0_name actuator1_name joint0_name joint1_name actuator0_serial actuator0_node actuator1_serial actuator1_node processor_firmware0 fpga_firmware0 processor_firmware1 fpga_firmware1" >
 	<Mechanism id="${mechanism_name}" type="complex">
 		<xacro:joint name="${joint0_name}" type="active"/>
 		<xacro:joint name="${joint1_name}" type="active"/>
 		<xacro:actuator name="${actuator0_name}" serial_number="${actuator0_serial}" node="${actuator0_node}" processor_firmware="${processor_firmware0}" fpga_firmware="${fpga_firmware0}"/>
-		<xacro:actuator name="${actuator1_name}" serial_number="${actuator1_serial}" node="${actuator1_node}" processor_firmware="${processor_firmware0}" fpga_firmware="${fpga_firmware0}"/>
+		<xacro:actuator name="${actuator1_name}" serial_number="${actuator1_serial}" node="${actuator1_node}" processor_firmware="${processor_firmware1}" fpga_firmware="${fpga_firmware1}"/>
 	</Mechanism>
 </xacro:macro>

Commit message: added FPGA string to applicable actuators

File: common/xacro/firmware/valkyrie_firmware.xacro (robot description, xacro)
@@ -21,25 +21,25 @@
     </xacro:macro>
     <xacro:property name="HipYawProcFirmware" value="${TurboProcRotaryFirmwareURL}" />
-    <xacro:property name="HipYawFPGAFirmware" value="" />
+    <xacro:property name="HipYawFPGAFirmware" value="${TurboFPGAFirmwareURL}" />
     <xacro:property name="HipRollProcFirmware" value="${TurboProcRotaryFirmwareURL}" />
-    <xacro:property name="HipRollFPGAFirmware" value="" />
+    <xacro:property name="HipRollFPGAFirmware" value="${TurboFPGAFirmwareURL}" />
     <xacro:property name="HipPitchProcFirmware" value="${TurboProcRotaryFirmwareURL}" />
-    <xacro:property name="HipPitchFPGAFirmware" value="" />
+    <xacro:property name="HipPitchFPGAFirmware" value="${TurboFPGAFirmwareURL}" />
     <xacro:property name="KneePitchProcFirmware" value="${TurboProcRotaryFirmwareURL}" />
-    <xacro:property name="KneePitchFPGAFirmware" value="" />
+    <xacro:property name="KneePitchFPGAFirmware" value="${TurboFPGAFirmwareURL}" />
     <xacro:property name="AnkleLeftActuatorProcFirmware" value="${TurboProcLinearFirmwareURL}" />
-    <xacro:property name="AnkleLeftActuatorFPGAFirmware" value="" />
+    <xacro:property name="AnkleLeftActuatorFPGAFirmware" value="${TurboFPGAFirmwareURL}" />
     <xacro:property name="AnkleRightActuatorProcFirmware" value="${TurboProcLinearFirmwareURL}" />
     <xacro:property name="AnkleRightActuatorFPGAFirmware" value="" />
     <xacro:property name="ShoulderPitchProcFirmware" value="${TurboProcRotaryFirmwareURL}" />
-    <xacro:property name="ShoulderPitchFPGAFirmware" value="" />
+    <xacro:property name="ShoulderPitchFPGAFirmware" value="${TurboFPGAFirmwareURL}" />
     <xacro:property name="ShoulderRollProcFirmware" value="${TurboProcRotaryFirmwareURL}" />
-    <xacro:property name="ShoulderRollFPGAFirmware" value="" />
+    <xacro:property name="ShoulderRollFPGAFirmware" value="${TurboFPGAFirmwareURL}" />
     <xacro:property name="ShoulderYawProcFirmware" value="${TurboProcRotaryFirmwareURL}" />
-    <xacro:property name="ShoulderYawFPGAFirmware" value="" />
+    <xacro:property name="ShoulderYawFPGAFirmware" value="${TurboFPGAFirmwareURL}" />
     <xacro:property name="ElbowPitchProcFirmware" value="${TurboProcRotaryFirmwareURL}" />
-    <xacro:property name="ElbowPitchFPGAFirmware" value="" />
-    <xacro:property name="ForearmYawProcFirmware" value="" />
-    <xacro:property name="ForearmYawFPGAFirmware" value="" />
+    <xacro:property name="ElbowPitchFPGAFirmware" value="${TurboFPGAFirmwareURL}" />
+    <xacro:property name="ForearmYawProcFirmware" value="${TurboFPGAFirmwareURL}" />
+    <xacro:property name="ForearmYawFPGAFirmware" value="${TurboFPGAFirmwareURL}" />
     <xacro:property name="LowerNeckPitchProcessorFirmware" value="" />
     <xacro:property name="LowerNeckPitchFPGAFirmware" value="" />
@@ -49,9 +49,9 @@
     <xacro:property name="UpperNeckPitchFPGAFirmware" value="" />
     <xacro:property name="TrunkYawProcessorFirmware" value="${TurboProcRotaryFirmwareURL}" />
-    <xacro:property name="TrunkYawFPGAFirmware" value="" />
+    <xacro:property name="TrunkYawFPGAFirmware" value="${TurboFPGAFirmwareURL}" />
     <xacro:property name="WaistRightActuatorProcessorFirmware" value="${TurboProcLinearFirmwareURL}" />
-    <xacro:property name="WaistRightActuatorFPGAFirmware" value="" />
+    <xacro:property name="WaistRightActuatorFPGAFirmware" value="${TurboFPGAFirmwareURL}" />
     <xacro:property name="WaistLeftActuatorProcessorFirmware" value="${TurboProcLinearFirmwareURL}" />
-    <xacro:property name="WaistLeftActuatorFPGAFirmware" value="" />
+    <xacro:property name="WaistLeftActuatorFPGAFirmware" value="${TurboFPGAFirmwareURL}" />
     <xacro:property name="leftForearmProcessorFirmware" value=""/>
     <xacro:property name="leftForearmFPGAFirmware" value=""/>
